File: ai03_PCB_guide.kicad_sch (KiCad schematic)
At the start: 10 parts

Commit message: finished MCU
Parts:
- added C? (x2): 22pF, symbol Device:C_Small
- added R?: R_Small, symbol Device:R_Small
- added SW?: SW_Push, symbol Switch:SW_Push
Connections:
- net +5V: now also R?.1
- net GND: now also Y?.2, Y?.4, C?.1, C?.1, SW?.1
- net at U?.17 (XTAL1), Y?.1: now also C?.2
- net at U?.16 (XTAL2), Y?.3: now also C?.2
- net D -: now reaches R?.1
- net D +: now reaches R?.1
- net at U?.13 (~{RESET}): now also R?.2, SW?.2

Commit message: finished schematic
Parts:
- added D1, D2, D3, D4: D_Small, Diode_SMD:D_SOD-123, symbol Device:D_Small
- added F1: 500mA, Fuse:Fuse_1206_3216Metric, symbol Device:Polyfuse
- added MX1, MX2, MX3, MX4: MX-NoLED, Button_Switch_Keyboard:SW_Cherry_MX_1.00u_PCB, symbol MX_Alps_Hybrid:MX-NoLED
- added USB1: Molex-0548190589, symbol random-keyboard-parts:Molex-0548190589
- C1, C2, C3, C4, C5, C6, C7: renamed from C?; footprint (none) -> Capacitor_SMD:C_0805_2012Metric
- R1: renamed from R?; footprint (none) -> Crystal:Crystal_SMD_3225-4Pin_3.2x2.5mm
- gave numbers to parts that had none: 6
Connections:
- net +5V: now also F1.2
- net D +: now also USB1.3 (D+)
- net D -: now also USB1.4 (D-)
- net GND: now also USB1.1 (GND)
- new net: D2.2 (A), MX2.2 (ROW)
- new net: D1.2 (A), MX1.2 (ROW)
- new net: D3.2 (A), MX3.2 (ROW)
- new net: D4.2 (A), MX4.2 (ROW)
- new net COL0: MX1.1 (COL), MX2.1 (COL)
- new net COL1: MX3.1 (COL), MX4.1 (COL)
- new net ROW0: D1.1 (K), D3.1 (K)
- new net ROW1: D2.1 (K), D4.1 (K)
- new net VCC: F1.1, USB1.5 (VBUS)

Commit message: added footprints to project
Parts:
- R1: footprint Crystal:Crystal_SMD_3225-4Pin_3.2x2.5mm -> Resistor_SMD:R_0805_2012Metric
- R2, R3, R4: footprint (none) -> Resistor_SMD:R_0805_2012Metric
Changed lines of the file:
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@@
 			)
 		)
-		(property "Footprint" ""
+		(property "Footprint" "Resistor_SMD:R_0805_2012Metric"
 			(at 111.76 31.75 0)
 			(effects
@@
 			)
 		)
-		(property "Footprint" ""
+		(property "Footprint" "Resistor_SMD:R_0805_2012Metric"
 			(at 154.94 91.44 0)
 			(effects
@@
 			)
 		)
-		(property "Footprint" "Crystal:Crystal_SMD_3225-4Pin_3.2x2.5mm"
+		(property "Footprint" "Resistor_SMD:R_0805_2012Metric"
 			(at 96.52 66.04 0)
 			(effects
@@
 			)
 		)
-		(property "Footprint" ""
+		(property "Footprint" "Resistor_SMD:R_0805_2012Metric"
 			(at 104.14 63.5 0)
 			(effects

Commit message: Added all footprints
Parts:
- MX1, MX2, MX3, MX4: footprint Button_Switch_Keyboard:SW_Cherry_MX_1.00u_PCB -> MX_Alps_Hybrid:MX-1U-NoLED
- SW1: footprint (none) -> random-keyboard-parts:SKQG-1155865
- USB1: footprint (none) -> random-keyboard-parts:Molex-0548190589
- Y1: footprint (none) -> Crystal:Crystal_SMD_3225-4Pin_3.2x2.5mm
Changed lines of the file:
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@@
 			)
 		)
-		(property "Footprint" ""
+		(property "Footprint" "random-keyboard-parts:Molex-0548190589"
 			(at 100.33 151.13 0)
 			(effects
@@
 			)
 		)
-		(property "Footprint" ""
+		(property "Footprint" "random-keyboard-parts:SKQG-1155865"
 			(at 105.41 33.02 0)
 			(effects
@@
 			)
 		)
-		(property "Footprint" "Button_Switch_Keyboard:SW_Cherry_MX_1.00u_PCB"
+		(property "Footprint" "MX_Alps_Hybrid:MX-1U-NoLED"
 			(at 186.055 98.425 0)
 			(effects
@@
 			)
 		)
-		(property "Footprint" "Button_Switch_Keyboard:SW_Cherry_MX_1.00u_PCB"
+		(property "Footprint" "MX_Alps_Hybrid:MX-1U-NoLED"
 			(at 202.565 97.155 0)
 			(effects
@@
 			)
 		)
-		(property "Footprint" "Button_Switch_Keyboard:SW_Cherry_MX_1.00u_PCB"
+		(property "Footprint" "MX_Alps_Hybrid:MX-1U-NoLED"
 			(at 186.055 80.645 0)
 			(effects
@@
 			)
 		)
-		(property "Footprint" ""
+		(property "Footprint" "Crystal:Crystal_SMD_3225-4Pin_3.2x2.5mm"
 			(at 101.6 45.72 0)
 			(effects
@@
 			)
 		)
-		(property "Footprint" "Button_Switch_Keyboard:SW_Cherry_MX_1.00u_PCB"
+		(property "Footprint" "MX_Alps_Hybrid:MX-1U-NoLED"
 			(at 202.565 80.645 0)
 			(effects
